File: src/juicePCB.kicad_pcb (KiCad board)
At the start: 2 copper layers, 61.6 x 99.4 mm, 12 parts, among them Q1 2N3904, SW1 SW_SPST

Commit message: Final rev.
Parts:
- moved D2 0.55 mm to (153.9, 85.0)
- renumbered KEYCHAIN to BOYKISSER
Routing:
- net +3V0: track 65.4 -> 66.1 mm
- net Net-(D2-K): track 33.9 -> 33.3 mm
